Commit message: feat: add gym2mujoco code architecture

File: assets/urdf/xarm6/xarm6_allegro_right_fsr_2023_thin_tilted.urdf (robot description, URDF)
Before this commit: robot xarm6, 47 links, 46 joints
Links:
- link base_link: geometry collision box size=0.0408 0.1130 0.095; visual box size=0.015 0.085 0.03
- link link1: geometry collision mesh filename=link1.stl; visual mesh filename=link1.stl
- link link2: geometry collision mesh filename=link2.stl; visual mesh filename=link2.stl
- link link3: geometry collision mesh filename=link3.stl; visual mesh filename=link3.stl
- link link4: geometry collision mesh filename=link4.stl; visual mesh filename=link4.stl
- link link5: geometry collision mesh filename=link5.stl; visual mesh filename=link5.stl
- link link6: geometry collision mesh filename=link6.stl; visual mesh filename=link6.stl
- link link_0.0: geometry collision box size=0.0196 0.0275 0.0164; visual mesh filename=link_0.0.STL
- link link_1.0: geometry collision box size=0.0196 0.0275 0.054; visual mesh filename=link_1.0.STL
- link link_10.0: geometry collision box size=0.0196 0.0275 0.0384; visual mesh filename=link_2.0.STL
- link link_11.0: geometry collision box size=0.0196 0.0275 0.02; visual mesh filename=link_3.0.STL
- link link_11.0_tip: geometry collision box size=0.014 0.014 0.04; visual mesh filename=modified_tip.STL scale=0.001 0.001 0.001
- link link_12.0: geometry collision box size=0.0358 0.034 0.0455; visual mesh filename=link_12.0_right.STL
- link link_13.0: geometry collision box size=0.0196 0.0275 0.0177; visual mesh filename=link_13.0.STL
- link link_14.0: geometry collision box size=0.0196 0.0275 0.0514; visual mesh filename=link_14.0.STL
- link link_15.0: geometry collision box size=0.0196 0.0275 0.034; visual mesh filename=link_15.0.STL
- link link_15.0_tip: geometry collision box size=0.014 0.014 0.04; visual mesh filename=modified_tip.STL scale=0.001 0.001 0.001
- link link_2.0: geometry collision box size=0.0196 0.0275 0.0384; visual mesh filename=link_2.0.STL
- link link_3.0: geometry collision box size=0.0196 0.0275 0.02; visual mesh filename=link_3.0.STL
- link link_3.0_tip: geometry collision box size=0.014 0.014 0.04; visual mesh filename=modified_tip.STL scale=0.001 0.001 0.001
- link link_4.0: geometry collision box size=0.0196 0.0275 0.0164; visual mesh filename=link_0.0.STL
- link link_5.0: geometry collision box size=0.0196 0.0275 0.054; visual mesh filename=link_1.0.STL
- link link_6.0: geometry collision box size=0.0196 0.0275 0.0384; visual mesh filename=link_2.0.STL
- link link_7.0: geometry collision box size=0.0196 0.0275 0.02; visual mesh filename=link_3.0.STL
- link link_7.0_tip: geometry collision box size=0.014 0.014 0.04; visual mesh filename=modified_tip.STL scale=0.001 0.001 0.001
- link link_8.0: geometry collision box size=0.0196 0.0275 0.0164; visual mesh filename=link_0.0.STL
- link link_9.0: geometry collision box size=0.0196 0.0275 0.054; visual mesh filename=link_1.0.STL
- link link_base: geometry collision mesh filename=base.stl; visual mesh filename=base.stl

Commit message: perf: add contact exclude for fsr in mujoco

File: assets/urdf/xarm6/xarm6_allegro_right_fsr_2023_thin_tilted.urdf (robot description, URDF)
Before this commit: robot xarm6, 47 links, 46 joints
Links:
- link base_link: geometry collision box size=0.0408 0.1130 0.095; visual box size=0.015 0.085 0.03
- link link_0.0: geometry collision box size=0.0196 0.0275 0.0164; visual mesh filename=link_0.0.obj
- link link_1.0: geometry collision box size=0.0196 0.0275 0.054; visual mesh filename=link_1.0.obj
- link link_10.0: geometry collision box size=0.0196 0.0275 0.0384; visual mesh filename=link_2.0.obj
- link link_11.0: geometry collision box size=0.0196 0.0275 0.02; visual mesh filename=link_3.0.obj
- link link_11.0_tip: geometry collision box size=0.014 0.014 0.04; visual mesh filename=modified_tip.obj scale=0.001 0.001 0.001
- link link_12.0: geometry collision box size=0.0358 0.034 0.0455; visual mesh filename=link_12.0_right.obj
- link link_13.0: geometry collision box size=0.0196 0.0275 0.0177; visual mesh filename=link_13.0.obj
- link link_14.0: geometry collision box size=0.0196 0.0275 0.0514; visual mesh filename=link_14.0.obj
- link link_15.0: geometry collision box size=0.0196 0.0275 0.034; visual mesh filename=link_15.0.obj
- link link_15.0_tip: geometry collision box size=0.014 0.014 0.04; visual mesh filename=modified_tip.obj scale=0.001 0.001 0.001
- link link_2.0: geometry collision box size=0.0196 0.0275 0.0384; visual mesh filename=link_2.0.obj
- link link_3.0: geometry collision box size=0.0196 0.0275 0.02; visual mesh filename=link_3.0.obj
- link link_3.0_tip: geometry collision box size=0.014 0.014 0.04; visual mesh filename=modified_tip.obj scale=0.001 0.001 0.001
- link link_4.0: geometry collision box size=0.0196 0.0275 0.0164; visual mesh filename=link_0.0.obj
- link link_5.0: geometry collision box size=0.0196 0.0275 0.054; visual mesh filename=link_1.0.obj
- link link_6.0: geometry collision box size=0.0196 0.0275 0.0384; visual mesh filename=link_2.0.obj
- link link_7.0: geometry collision box size=0.0196 0.0275 0.02; visual mesh filename=link_3.0.obj
- link link_7.0_tip: geometry collision box size=0.014 0.014 0.04; visual mesh filename=modified_tip.obj scale=0.001 0.001 0.001
- link link_8.0: geometry collision box size=0.0196 0.0275 0.0164; visual mesh filename=link_0.0.obj
- link link_9.0: geometry collision box size=0.0196 0.0275 0.054; visual mesh filename=link_1.0.obj
